File: RAK811_LORA_ADAPTABLE_NODE.kicad_pcb (KiCad board)
At the start: 2 copper layers, 75 x 49 mm, 18 parts, among them J1 Screw_Terminal_01x02, J2 Screw_Terminal_01x03, J3 Conn_01x01_Male, J4 Conn_01x01_Male, J5 Conn_01x01_Male, J6 Conn_01x01_Male, J7 Conn_Coaxial, U1 RAK811-HF

Commit message: some i/o pins layout
Parts:
- removed H1, H6: MountingHole, MountingHole:MountingHole_3mm
- added J10: Conn_01x01_Male, Connector_Wire:SolderWirePad_1x01_Drill0.8mm, F.Cu at (137.1, 124.4)
- added J11: Conn_01x01_Male, Connector_Wire:SolderWirePad_1x01_Drill0.8mm, F.Cu at (162.5, 129.5)
- added J12: Conn_01x01_Male, Connector_Wire:SolderWirePad_1x01_Drill0.8mm, F.Cu at (137.1, 119.3)
- added J13: Conn_01x01_Male, Connector_Wire:SolderWirePad_1x01_Drill0.8mm, F.Cu at (137.1, 127.0)
- added J14: Conn_01x01_Male, Connector_Wire:SolderWirePad_1x01_Drill0.8mm, F.Cu at (162.5, 119.3)
- added J15: Conn_01x01_Male, Connector_Wire:SolderWirePad_1x01_Drill0.8mm, F.Cu at (139.6, 119.3)
- added J8: Conn_01x01_Male, Connector_Wire:SolderWirePad_1x01_Drill0.8mm, F.Cu at (137.1, 121.9)
- added J9: Conn_01x01_Male, Connector_Wire:SolderWirePad_1x01_Drill0.8mm, F.Cu at (137.1, 129.5)
- moved BT1 52.1 mm to (109.2, 108.6), turned to 0 degrees
- moved BT2 52.1 mm to (161.3, 140.3), turned to 180 degrees
- moved JP1 35.0 mm to (132.1, 102.9)
- moved J4 25.8 mm to (167.0, 148.0)
- moved J5 24.7 mm to (184.2, 131.4)
- moved J3 19.6 mm to (167.0, 144.8)
- moved J7 1.27 mm to (102.2, 118.1)
- moved JP2 1.27 mm to (107.3, 118.7)
- moved J2 0.90 mm to (168.9, 140.3)
- moved J1 0.90 mm to (168.9, 113.0)
- moved J6 0.90 mm to (102.9, 111.1)
Connections:
- J1 pad 1: Net-(J1-Pad1) -> Net-(BT2-Pad2)
- J1 pad 2: Net-(BT2-Pad2) -> Net-(J1-Pad2)
- JP1 pad 2: Net-(J1-Pad1) -> Net-(J1-Pad2)
- U1 pad 11: Net-(J1-Pad1) -> Net-(J1-Pad2)
Routing:
- net Net-(BT2-Pad2): track 0.00 -> 141.3 mm
- net Net-(J1-Pad2): track 0.00 -> 59.4 mm
- net Net-(BT1-Pad2): track 0.00 -> 30.2 mm
- net Net-(BT1-Pad1): track 0.00 -> 23.9 mm
- net Net-(J6-Pad1): track 0.00 -> 8.92 mm
- net Net-(JP2-Pad2): track 0.00 -> 7.74 mm
- net Net-(J7-Pad1): track 0.00 -> 4.83 mm

Commit message: half i/o pins layout
Parts:
- added J16: Conn_01x01_Male, Connector_Wire:SolderWirePad_1x01_Drill0.8mm, F.Cu at (154.9, 119.3)
- added J17: Conn_01x01_Male, Connector_Wire:SolderWirePad_1x01_Drill0.8mm, F.Cu at (152.3, 119.3)
- added J18: Conn_01x01_Male, Connector_Wire:SolderWirePad_1x01_Drill0.8mm, F.Cu at (149.8, 119.3)
- added J19: Conn_01x01_Male, Connector_Wire:SolderWirePad_1x01_Drill0.8mm, F.Cu at (147.3, 119.3)
- added J20: Conn_01x01_Male, Connector_Wire:SolderWirePad_1x01_Drill0.8mm, F.Cu at (142.2, 119.3)
- added J21: Conn_01x01_Male, Connector_Wire:SolderWirePad_1x01_Drill0.8mm, F.Cu at (144.7, 119.3)
- added J22: Conn_01x01_Male, Connector_Wire:SolderWirePad_1x01_Drill0.8mm, F.Cu at (160.0, 119.3)
- added J23: Conn_01x01_Male, Connector_Wire:SolderWirePad_1x01_Drill0.8mm, F.Cu at (157.4, 119.3)

Commit message: all i/o pins layout
Parts:
- added J24: Conn_01x01_Male, Connector_Wire:SolderWirePad_1x01_Drill0.8mm, F.Cu at (152.3, 129.5)
- added J25: Conn_01x01_Male, Connector_Wire:SolderWirePad_1x01_Drill0.8mm, F.Cu at (149.8, 129.5)
- added J26: Conn_01x01_Male, Connector_Wire:SolderWirePad_1x01_Drill0.8mm, F.Cu at (147.3, 129.5)
- added J27: Conn_01x01_Male, Connector_Wire:SolderWirePad_1x01_Drill0.8mm, F.Cu at (154.9, 129.5)
- added J28: Conn_01x01_Male, Connector_Wire:SolderWirePad_1x01_Drill0.8mm, F.Cu at (139.6, 129.5)
- added J29: Conn_01x01_Male, Connector_Wire:SolderWirePad_1x01_Drill0.8mm, F.Cu at (142.2, 129.5)
- added J30: Conn_01x01_Male, Connector_Wire:SolderWirePad_1x01_Drill0.8mm, F.Cu at (144.7, 129.5)
- added J31: Conn_01x01_Male, Connector_Wire:SolderWirePad_1x01_Drill0.8mm, F.Cu at (157.4, 129.5)
- added J32: Conn_01x01_Male, Connector_Wire:SolderWirePad_1x01_Drill0.8mm, F.Cu at (160.0, 129.5)
- moved J4 24.0 mm to (162.5, 124.4)
- moved J5 23.7 mm to (162.5, 121.9)
- moved J3 18.4 mm to (162.5, 127.0)
Other:
- board text added: "RAK811 LORA ADAPTABLE NODE"
