File: RAK811_LORA_ADAPTABLE_NODE.kicad_pcb (KiCad board)
At the start: 2 copper layers, 75 x 49 mm, 23 parts, among them J1 Screw_Terminal_01x03, J10 Conn_01x09_Male, J11 Conn_01x09_Male, J12 Conn_01x09_Male, J2 Screw_Terminal_01x03, J3 Conn_01x03_Male, J4 Conn_01x03_Male, J5 Conn_01x11_Male, J6 Conn_01x01_Male, J7 Conn_Coaxial, J8 Conn_01x11_Male, J9 Conn_01x01_Male, U1 RAK811-HF

Commit message: fine tuned routing
Parts:
- moved BT1 0.50 mm to (109.2, 109.1)
- moved BT2 0.42 mm to (161.3, 139.9)
Routing:
- net Net-(J8-Pad1): track 64.1 -> 65.9 mm
- net Net-(J8-Pad2): track 60.0 -> 61.0 mm
- net Net-(BT1-Pad1): track 24.8 -> 25.5 mm
- net Net-(J1-Pad3): track 69.9 -> 69.3 mm
- net Net-(J8-Pad7): track 28.4 -> 28.9 mm
- net Net-(J8-Pad4): track 44.8 -> 45.3 mm
- net Net-(J8-Pad3): track 50.5 -> 51.0 mm
- net Net-(J8-Pad6): track 33.9 -> 34.4 mm
- net Net-(J8-Pad5): track 39.3 -> 39.9 mm
